File: kicad/euclid-16.kicad_sch (KiCad schematic)
At the start: 46 parts, among them J1 MIDI sync in, J2 Audio out, SW1 SW_Push, SW2 SW_Push, SW3 SW_Push, SW4 SW_Push, SW5 RotaryEncoder_Switch, U1 74HC595, U2 74HC595

Commit message: fix 3.3v ref
Parts:
- R18: value 4.7k -> 1k
Connections:
- net +3.3V: now reaches A1.36 (3V3)
- net +3.3V: now also U1.10 (~{SRCLR}), U1.16 (VCC), U2.10 (~{SRCLR}), U2.16 (VCC)
- removed net +5V: A1.40 (VBUS), U1.10 (~{SRCLR}), U1.16 (VCC), U2.10 (~{SRCLR}), U2.16 (VCC)

Commit message: fix clock in
Parts:
- J1: value MIDI sync in -> Clock IN
- J2: value Audio out -> Audio OUT
Connections:
- net midi_clkin renamed clock_in
Changed lines of the file:
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@@
 		)
 	)
-	(global_label "midi_clkin"
+	(global_label "clock_in"
 		(shape input)
 		(at 93.98 91.44 270)
@@
 		)
 		(property "Intersheetrefs" "${INTERSHEET_REFS}"
-			(at 93.98 103.9804 90)
+			(at 93.98 102.1661 90)
 			(effects
 				(font
@@
 		)
 	)
-	(global_label "midi_clkin"
+	(global_label "clock_in"
 		(shape input)
 		(at 245.11 76.2 180)
@@
 		)
 		(property "Intersheetrefs" "${INTERSHEET_REFS}"
-			(at 232.5696 76.2 0)
+			(at 234.3839 76.2 0)
 			(effects
 				(font
@@
 			)
 		)
-		(property "Value" "MIDI sync in"
+		(property "Value" "Clock IN"
 			(at 255.27 78.1049 0)
 			(effects
@@
 			)
 		)
-		(property "Value" "Audio out"
+		(property "Value" "Audio OUT"
 			(at 255.27 98.4249 0)
 			(effects

Commit message: update sch
Parts:
- removed 100nF1: C, Capacitor_THT:C_Disc_D3.0mm_W1.6mm_P2.50mm, symbol Device:C
- added C1: 100nF, symbol Device:C
- added C2: 47nF, symbol Device:C
- added R17: 220, Resistor_THT:R_Axial_DIN0207_L6.3mm_D2.5mm_P7.62mm_Horizontal, symbol Device:R_US
- added R20: 20k, Resistor_THT:R_Axial_DIN0207_L6.3mm_D2.5mm_P7.62mm_Horizontal, symbol Device:R_US
- added R21: 1.8k, Resistor_THT:R_Axial_DIN0207_L6.3mm_D2.5mm_P7.62mm_Horizontal, symbol Device:R_US
- added R22: 10k, Resistor_THT:R_Axial_DIN0207_L6.3mm_D2.5mm_P7.62mm_Horizontal, symbol Device:R_US
- J1: value Clock IN -> Clock IN (4 PPQN)
- R19: renamed from R18; value 1k -> 100
- renumbered R17 to R18
Connections:
- net GND: now also R19.2, C1.2, R20.2, R21.2
- net clock_in: now also A1.17 (GPIO13), R20.1, R22.1; no longer A1.16 (GPIO12), J1.T
- net enc_A: now also A1.22 (GPIO17); no longer A1.21 (GPIO16)
- net enc_B: now also A1.21 (GPIO16); no longer A1.22 (GPIO17)
- net pwm_out: now also A1.20 (GPIO15), R17.1; no longer R19.2
- net at J2.T: now also C2.2, R21.1; no longer R19.1
- net +3.3V renamed 3.3V
- new net: J1.T, R22.2
- new net: C1.1, C2.1, R17.2, R19.1
Other:
- moved on the sheet: J2, R19
